File: plug-ins/hard/RPSPMC/CAD/rpZ7020_adda_io_shield/rpZ7020_adda_io_shield.kicad_pcb (KiCad board)
At the start: 4 copper layers, 70.6 x 94.5 mm, 36 parts, among them J1 Samtec_ASP-134486-01, J2 Conn_01x03_Socket, J2-FMC-RP1 Conn_02x20, J2-PWR3 Conn_01x03_Pin, J3-FMC-POWER1 Conn_02x06_Odd_Even, J3-PWR12 Conn_01x02_Pin, J4-FMC-AUX1 Conn_02x06_Odd_Even

Commit message: last tweaks before order rev 1.0.1 PCB
Connections:
- J2-FMC-RP1 pad 33: unconnected-(J2-FMC-RP1-Pin_33-Pad33) -> VADJ
Routing:
- net VADJ: track 45.3 -> 49.7 mm
- net D2P RP: track 70.0 -> 68.4 mm
